Commit message: Separate starting of controllers to simplify multi-robot structure. Add direct names of the controllers for the robot. Base example: working all 3.

File: hercules_description/urdf/hercules.urdf.xacro (robot description, xacro)
@@ -4,156 +4,19 @@
    <xacro:arg name="name" default="hercules"/>
    <xacro:arg name="prefix" default="" />
-   <!-- parameters -->
-   <xacro:arg name="prefix" default="" />
-   <xacro:arg name="joint_limit_params" default=""/>
-   <xacro:arg name="kinematics_params" default=""/>
-   <xacro:arg name="physical_params" default=""/>
-   <xacro:arg name="visual_params" default=""/>
-   <xacro:arg name="transmission_hw_interface" default=""/>
-   <xacro:arg name="safety_limits" default="false"/>
-   <xacro:arg name="safety_pos_margin" default="0.15"/>
-   <xacro:arg name="safety_k_position" default="20"/>
    <!-- ros2_control related parameters -->
    <xacro:arg name="use_mock_hardware" default="true" />
    <xacro:arg name="mock_sensor_commands" default="false" />
-   <xacro:arg name="headless_mode" default="false" />
-   <!-- initial position for fake hardware -->
-   <xacro:arg name="initial_positions_port_file" default="$(find hercules_description)/config/initial_positions_port_arm.yaml"/>
-   <xacro:arg name="initial_positions_starboard_file" default="$(find hercules_description)/config/initial_positions_starboard_arm.yaml"/>
    <!-- Simulation parameter -->
    <xacro:arg name="sim_gazebo_classic" default="false" />
    <xacro:arg name="sim_gazebo" default="false" />
-   <xacro:arg name="simulation_controllers" default="$(find hercules_description)/config/hercules_controllers.yaml" />
    <!-- import Husky macro -->
-   <xacro:include filename="$(find husky_description)/urdf/husky_macro.urdf.xacro"/>
-   <!-- import UR macro -->
-   <xacro:include filename="$(find ur_description)/urdf/ur_macro.xacro"/>
-   <!-- import gripper macro -->
-   <xacro:include filename="$(find robotiq_85_description)/urdf/robotiq_85_gripper_macro.urdf.xacro" />
-   <!-- UR parameters -->
-   <xacro:arg name="prefix" default="" />
-   <xacro:arg name="joint_limit_params" default=""/>
-   <xacro:arg name="kinematics_params" default=""/>
-   <xacro:arg name="physical_params" default=""/>
-   <xacro:arg name="visual_params" default=""/>
-   <xacro:arg name="transmission_hw_interface" default=""/>
-   <xacro:arg name="safety_limits" default="false"/>
-   <xacro:arg name="safety_pos_margin" default="0.15"/>
-   <xacro:arg name="safety_k_position" default="20"/>
-   <!-- convert to property to use substitution in function -->
-   <xacro:property name="initial_positions_port_file" default="$(arg initial_positions_port_file)"/>
-   <xacro:property name="initial_positions_starboard_file" default="$(arg initial_positions_starboard_file)"/>
-   <!-- Load husky description -->
-   <xacro:husky
+   <xacro:include filename="$(find hercules_description)/urdf/hercules_macro.urdf.xacro"/>
+   <!-- Load hercules description -->
+   <xacro:hercules
      prefix="$(arg prefix)"
-     is_sim="$(arg sim_gazebo_classic)"
-     use_mock_hardware="$(arg use_mock_hardware)"
-    />
-   <xacro:property name="box_base_size" value="0.3" />
-   <!-- Add Fixture links for manipulators -->
-   <link name="$(arg prefix)manipulator_fixture_box">
-     <visual>
-       <origin xyz="0 0 0" rpy="0 0 0"/>
-       <geometry>
-         <box size="${box_base_size} ${box_base_size} ${box_base_size}"/>
-       </geometry>
-       <material name="sr_violet">
-         <color rgba="${102/255} ${46/255} ${145/255} 1.0" />
-       </material>
-     </visual>
-     <collision>
-       <origin xyz="0 0 0" rpy="0 0 0"/>
-       <geometry>
-         <box size="${box_base_size} ${box_base_size} ${box_base_size}"/>
-       </geometry>
-     </collision>
-   </link>
-   <joint name="$(arg prefix)base_link-$(arg prefix)manipulator_fixture_box" type="fixed">
-     <parent link="$(arg prefix)base_link" />
-     <child link="$(arg prefix)manipulator_fixture_box" />
-     <origin xyz="0 0 ${ box_base_size/2 + 0.245 }" rpy="0 0 0" />
-   </joint>
-   <!-- arm -->
-   <xacro:ur_robot
-     name="$(arg prefix)port_$(arg name)"
-     tf_prefix="$(arg prefix)port_"
-     parent="$(arg prefix)manipulator_fixture_box"
-     joint_limits_parameters_file="$(arg joint_limit_params)"
-     kinematics_parameters_file="$(arg kinematics_params)"
-     physical_parameters_file="$(arg physical_params)"
-     visual_parameters_file="$(arg visual_params)"
-     transmission_hw_interface="$(arg transmission_hw_interface)"
-     safety_limits="$(arg safety_limits)"
-     safety_pos_margin="$(arg safety_pos_margin)"
-     safety_k_position="$(arg safety_k_position)"
-     use_mock_hardware="$(arg use_mock_hardware)"
-     mock_sensor_commands="$(arg mock_sensor_commands)"
-     headless_mode="$(arg headless_mode)"
-     initial_positions="${xacro.load_yaml(initial_positions_port_file)}"
-     sim_gazebo_classic="$(arg sim_gazebo_classic)"
-     sim_gazebo="$(arg sim_gazebo)" >
-     <origin xyz="0 ${ box_base_size/2 } 0" rpy="${pi/2} 0 ${pi}" />          <!-- position robot in the world -->
-   </xacro:ur_robot>
-   <xacro:robotiq_85_gripper
-     name="$(arg prefix)port_gripper_$(arg name)"
-     prefix="$(arg prefix)port_"
-     parent="$(arg prefix)port_tool0"
      use_mock_hardware="$(arg use_mock_hardware)"
      mock_sensor_commands="$(arg mock_sensor_commands)"
      sim_gazebo_classic="$(arg sim_gazebo_classic)"
-     sim_gazebo="$(arg sim_gazebo)" >
-     <origin xyz="0 0 0" rpy="0 -${pi/2} 0"/>
-   </xacro:robotiq_85_gripper>
-   <!-- arm -->
-   <xacro:ur_robot
-     name="$(arg prefix)starboard_$(arg name)"
-     tf_prefix="$(arg prefix)starboard_"
-     parent="$(arg prefix)manipulator_fixture_box"
-     joint_limits_parameters_file="$(arg joint_limit_params)"
-     kinematics_parameters_file="$(arg kinematics_params)"
-     physical_parameters_file="$(arg physical_params)"
-     visual_parameters_file="$(arg visual_params)"
-     transmission_hw_interface="$(arg transmission_hw_interface)"
-     safety_limits="$(arg safety_limits)"
-     safety_pos_margin="$(arg safety_pos_margin)"
-     safety_k_position="$(arg safety_k_position)"
-     use_mock_hardware="$(arg use_mock_hardware)"
-     mock_sensor_commands="$(arg mock_sensor_commands)"
-     headless_mode="$(arg headless_mode)"
-     initial_positions="${xacro.load_yaml(initial_positions_starboard_file)}"
-     sim_gazebo_classic="$(arg sim_gazebo_classic)"
-     sim_gazebo="$(arg sim_gazebo)" >
-     <origin xyz="0 -${ box_base_size/2 } 0" rpy="${pi/2} 0 0" />          <!-- position robot in the world -->
-   </xacro:ur_robot>
-   <xacro:robotiq_85_gripper
-     name="$(arg prefix)starboard_gripper_$(arg name)"
-     prefix="$(arg prefix)starboard_"
-     parent="$(arg prefix)starboard_tool0"
-     use_mock_hardware="$(arg use_mock_hardware)"
-     mock_sensor_commands="$(arg mock_sensor_commands)"
-     sim_gazebo_classic="$(arg sim_gazebo_classic)"
-     sim_gazebo="$(arg sim_gazebo)">
-     <origin xyz="0 0 0" rpy="0 -${pi/2} 0"/>
-   </xacro:robotiq_85_gripper>
-   <xacro:if value="$(arg sim_gazebo_classic)">
-     <!-- Gazebo plugins -->
-     <gazebo reference="world">
-     </gazebo>
-     <gazebo>
-       <plugin filename="libgazebo_ros2_control.so" name="gazebo_ros2_control">
-         <parameters>$(arg simulation_controllers)</parameters>
-       </plugin>
-     </gazebo>
-   </xacro:if>
-   <xacro:if value="$(arg sim_gazebo)">
-     <!-- Ignition plugins -->
-     <gazebo reference="world">
-     </gazebo>
-     <gazebo>
-       <plugin filename="libignition_ros2_control-system.so" name="ignition_ros2_control::IgnitionROS2ControlPlugin">
-         <parameters>$(arg simulation_controllers)</parameters>
-         <controller_manager_node_name>$(arg prefix)controller_manager</controller_manager_node_name>
-       </plugin>
-     </gazebo>
-   </xacro:if>
+     sim_gazebo="$(arg sim_gazebo)"
+    />
 </robot>
