Commit message: remove suspension joints

File: tiago_chaining/config/tiago_full_unrolled.urdf (robot description, URDF)
Before this commit: robot tiago, 54 links, 53 joints
Links:
- removed link suspension_left_link
- removed link suspension_right_link
Joints:
- removed joint suspension_left_joint
- removed joint suspension_right_joint
- joint wheel_left_joint: parent suspension_left_link -> base_link
- joint wheel_right_joint: parent suspension_right_link -> base_link
